File: schematic/audio-prototype-board/audio-prototype-board.kicad_pcb (KiCad board)
At the start: 2 copper layers, 261.6 x 132.1 mm, 9 parts, among them IC1 TC1044SCPA, IC2 TC1044SCPA, IC3 TC1044SCPA, IC4 L7805CV, IC5 L7809CV, IC6 L7812CV, J1 163-179PH-EX

Commit message: Made a footprint for the carrier boards. Test placed it on the PCB.
Parts:
- added REF**: Potentiometer Carrier Board 24mm, Ivan Hawkes:Potentiometer Carrier Board 24mm, F.Cu at (119.4, 50.8)
- added REF**: Potentiometer Carrier Board 24mm, Ivan Hawkes:Potentiometer Carrier Board 24mm, F.Cu at (233.7, 50.8)
- added REF**: Potentiometer Carrier Board 24mm, Ivan Hawkes:Potentiometer Carrier Board 24mm, F.Cu at (157.5, 50.8)
- added REF**: Potentiometer Carrier Board 24mm, Ivan Hawkes:Potentiometer Carrier Board 24mm, F.Cu at (195.6, 50.8)
- added REF**: Potentiometer Carrier Board 24mm, Ivan Hawkes:Potentiometer Carrier Board 24mm, F.Cu at (81.3, 50.8)
- added REF**: Potentiometer Carrier Board 24mm, Ivan Hawkes:Potentiometer Carrier Board 24mm, F.Cu at (43.2, 50.8)
- moved IC1 118.6 mm to (153.7, 128.3)
- moved IC2 118.6 mm to (179.1, 130.8)
- moved IC3 118.6 mm to (196.8, 128.3)
- moved IC5 26.0 mm to (238.7, 116.8)
- moved IC4 26.0 mm to (203.2, 116.8)
- moved IC6 26.0 mm to (221.0, 116.8)
- moved C1 26.0 mm to (249.0, 88.9)
- moved J1 26.0 mm to (270.1, 103.0)
- moved D1 26.0 mm to (246.4, 101.6)

Commit message: Resized the page.
Parts:
- moved REF** 19.3 mm to (137.2, 43.2)
- moved REF** 19.3 mm to (251.5, 43.2)
- moved REF** 19.3 mm to (175.3, 43.2)
- moved REF** 19.3 mm to (213.4, 43.2)
- moved REF** 19.3 mm to (99.1, 43.2)
- moved REF** 19.3 mm to (61.0, 43.2)
Other:
- board size 261.6 x 132.1 mm -> 297.2 x 210.8 mm
Changed lines of the file:
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@@
     (thickness 1.6)
   )
-  (paper "A4")
+  (paper "A3")
   (layers
     (0 "F.Cu" signal)
@@
   )
   (footprint "Ivan Hawkes:Potentiometer Carrier Board 24mm" (layer "F.Cu")
-    (at 119.38 50.8)
+    (at 137.16 43.18)
     (attr through_hole)
     (fp_text reference "REF**" (at 0 -0.5 unlocked) (layer "F.SilkS")
@@
   )
   (footprint "Ivan Hawkes:Potentiometer Carrier Board 24mm" (layer "F.Cu")
-    (at 233.68 50.8)
+    (at 251.46 43.18)
     (attr through_hole)
     (fp_text reference "REF**" (at 0 -0.5 unlocked) (layer "F.SilkS")
@@
         (effects (font (size 1 1) (thickness 0.15)))
     )
+    (fp_text user "${REFERENCE}" (at 15.24 5.08 90) (layer "F.Fab")
+        (effects (font (size 1 1) (thickness 0.15)))
+    )
+    (fp_text user "${REFERENCE}" (at 0 2.5 unlocked) (layer "F.Fab")
+        (effects (font (size 1 1) (thickness 0.15)))
+    )
     (fp_text user "${REFERENCE}" (at -15.24 5.08 90) (layer "F.Fab")
-        (effects (font (size 1 1) (thickness 0.15)))
-    )
-    (fp_text user "${REFERENCE}" (at 15.24 5.08 90) (layer "F.Fab")
-        (effects (font (size 1 1) (thickness 0.15)))
-    )
-    (fp_text user "${REFERENCE}" (at 0 2.5 unlocked) (layer "F.Fab")
         (effects (font (size 1 1) (thickness 0.15)))
     )
@@
   )
   (footprint "Ivan Hawkes:Potentiometer Carrier Board 24mm" (layer "F.Cu")
-    (at 157.48 50.8)
+    (at 175.26 43.18)
     (attr through_hole)
     (fp_text reference "REF**" (at 0 -0.5 unlocked) (layer "F.SilkS")
@@
   )
   (footprint "Ivan Hawkes:Potentiometer Carrier Board 24mm" (layer "F.Cu")
-    (at 195.58 50.8)
+    (at 213.36 43.18)
     (attr through_hole)
     (fp_text reference "REF**" (at 0 -0.5 unlocked) (layer "F.SilkS")
@@
         (effects (font (size 1 1) (thickness 0.15)))
     )
+    (fp_text user "${REFERENCE}" (at 0 2.5 unlocked) (layer "F.Fab")
+        (effects (font (size 1 1) (thickness 0.15)))
+    )
     (fp_text user "${REFERENCE}" (at -15.24 5.08 90) (layer "F.Fab")
         (effects (font (size 1 1) (thickness 0.15)))
     )
     (fp_text user "${REFERENCE}" (at 15.24 5.08 90) (layer "F.Fab")
-        (effects (font (size 1 1) (thickness 0.15)))
-    )
-    (fp_text user "${REFERENCE}" (at 0 2.5 unlocked) (layer "F.Fab")
         (effects (font (size 1 1) (thickness 0.15)))
     )
@@
   )
   (footprint "Ivan Hawkes:Potentiometer Carrier Board 24mm" (layer "F.Cu")
-    (at 81.28 50.8)
+    (at 99.06 43.18)
     (attr through_hole)
     (fp_text reference "REF**" (at 0 -0.5 unlocked) (layer "F.SilkS")
@@
         (effects (font (size 1 1) (thickness 0.15)))
     )
+    (fp_text user "${REFERENCE}" (at 0 2.5 unlocked) (layer "F.Fab")
+        (effects (font (size 1 1) (thickness 0.15)))
+    )
     (fp_text user "${REFERENCE}" (at 15.24 5.08 90) (layer "F.Fab")
-        (effects (font (size 1 1) (thickness 0.15)))
-    )
-    (fp_text user "${REFERENCE}" (at 0 2.5 unlocked) (layer "F.Fab")
         (effects (font (size 1 1) (thickness 0.15)))
     )
@@
   )
   (footprint "Ivan Hawkes:Potentiometer Carrier Board 24mm" (layer "F.Cu")
-    (at 43.18 50.8)
+    (at 60.96 43.18)
     (attr through_hole)
     (fp_text reference "REF**" (at 0 -0.5 unlocked) (layer "F.SilkS")
@@
         (effects (font (size 1 1) (thickness 0.15)))
     )
+    (fp_text user "${REFERENCE}" (at 0 2.5 unlocked) (layer "F.Fab")
+        (effects (font (size 1 1) (thickness 0.15)))
+    )
+    (fp_text user "${REFERENCE}" (at 15.24 5.08 90) (layer "F.Fab")
+        (effects (font (size 1 1) (thickness 0.15)))
+    )
     (fp_text user "${REFERENCE}" (at -15.24 5.08 90) (layer "F.Fab")
-        (effects (font (size 1 1) (thickness 0.15)))
-    )
-    (fp_text user "${REFERENCE}" (at 15.24 5.08 90) (layer "F.Fab")
-        (effects (font (size 1 1) (thickness 0.15)))
-    )
-    (fp_text user "${REFERENCE}" (at 0 2.5 unlocked) (layer "F.Fab")
         (effects (font (size 1 1) (thickness 0.15)))
     )
@@
     )
   )
-  (gr_rect (start 17.78 25.4) (end 279.4 157.48)
+  (gr_rect (start 20.32 20.32) (end 317.5 231.14)
     (stroke (width 0.1) (type default)) (fill none) (layer "Edge.Cuts"))
 )
